File: DCmotors+driver.brd (EAGLE design)
At the start: 68.6 x 53.3 mm, 7 parts

Commit message: Add files via upload
Parts:
- removed U3: (no value), AUTODESK_CIRCUITS_BREADBOARD:DIL16
- added U1: (no value), AUTODESK_CIRCUITS_BREADBOARD:ARDUINO_UNO
- S1: device AUTODESK_CIRCUITS_BREADBOARD:TL1105 -> AUTODESK_CIRCUITS_BREADBOARD:M251
- U2: device AUTODESK_CIRCUITS_BREADBOARD:ARDUINO_UNO -> AUTODESK_CIRCUITS_BREADBOARD:DIL16
- moved U2 12.7 mm to (5.00, 35.5)
- renumbered S2 to S3
Connections:
- removed net N$17: BAT1.-, S1.3, S3.1, U2.GND., U3.13, U3.4
- removed net N$18: BAT1.+, S3.3, U3.16, U3.8
- net N$1: now also BAT1.+, S1.3, S3.3, U2.16, U2.8; no longer U2.9, U3.1
- net N$10: now also U1.3, U2.9; no longer U3.12
- net N$11: now also U1.5, U2.10; no longer M1.1, U3.14
- net N$12: now also M1.2, U2.11; no longer U2.4, U3.15
- net N$13: now also U2.12; no longer S1.4, U2.2
- net N$14: now also M1.1, U2.14; no longer S1.2
- net N$15: now also U1.4, U2.15; no longer S1.1
- net N$16: now also U1.2; no longer U2.12
- net N$2: now also S1.2, U1.12; no longer U2.8, U3.2
- net N$3: now also U1.9, U2.1; no longer M2.2, U3.3
- net N$4: now also U1.8, U2.2; no longer U3.5
- net N$5: now also M2.2, U2.3; no longer M2.1, U3.6
- net N$6: now also BAT1.-, S1.1, S3.1, U1.GND., U2.13, U2.4; no longer U2.7, U3.7
- net N$7: now also U2.5; no longer U2.3, U3.9
- net N$8: now also M2.1, U2.6; no longer U2.5, U3.10
- net N$9: now also U1.7, U2.7; no longer M1.2, U3.11
